Commit message: first try of corespondance grouping

File: simulation_tobot/URDF/tobot.urdf.xacro (robot description, xacro)
@@ -157,5 +157,5 @@
   </joint>
   <!--CAMERA-->
-  <link name="camera">
+  <link name="camera_link">
     <visual>
       <geometry>
@@ -166,7 +166,7 @@
     </visual>
   </link>
-  <joint name="camera" type="fixed">
+  <joint name="camera_link" type="fixed">
     <parent link="base_link"/>
-    <child link="camera"/>
+    <child link="camera_link"/>
     <origin xyz="${width} 0 ${GROUND_CLEARANCE-bodylen+posz_camera} " rpy="${-PI/2} 0 ${-PI/2}"/>
   </joint>

Commit message: Launch file for simulation with two robots and some parameters file for arbotix simulation

File: simulation_tobot/URDF/tobot.urdf.xacro (robot description, xacro)
@@ -14,4 +14,5 @@
   <xacro:property name="fwheel_rad" value="0.0325" />
   <xacro:property name="PI" value="3.1415" />
+  <xacro:property name="prefix" value="" />
   <material name="black">
     <color rgba="0 0 0 1"/>
@@ -21,5 +22,5 @@
   </material>
   <!-- Actual frame and materials -->
-  <link name="base_link">
+  <link name="${prefix}base_link">
     <visual>
       <geometry>
@@ -38,5 +39,5 @@
     </collision>
   </link>
-  <link name="lwheel">
+  <link name="${prefix}lwheel">
     <visual>
       <geometry>
@@ -53,11 +54,11 @@
     </collsion>
   </link>
-  <joint name="base_to_lwheel" type="continuous">
-    <parent link="base_link"/>
-    <child link="lwheel"/>
+  <joint name="${prefix}base_to_lwheel" type="continuous">
+    <parent link="${prefix}base_link"/>
+    <child link="${prefix}lwheel"/>
     <axis xyz="0 1 0"/>
     <origin xyz="0 ${width} ${GROUND_CLEARANCE-(bodylen/2)}" rpy="0 0 0"/>
   </joint>
-  <link name="rwheel">
+  <link name="${prefix}rwheel">
     <visual>
       <geometry>
@@ -74,12 +75,12 @@
     </collsion>
   </link>
-  <joint name="base_to_rwheel" type="continuous">
-    <parent link="base_link"/>
-    <child link="rwheel"/>
+  <joint name="${prefix}base_to_rwheel" type="continuous">
+    <parent link="${prefix}base_link"/>
+    <child link="${prefix}rwheel"/>
     <axis xyz="0 1 0"/>
     <origin xyz="0 ${-width} ${GROUND_CLEARANCE-(bodylen/2)}" rpy="0 0 0"/>
   </joint>
   <!--LASER-->
-  <link name="laser">
+  <link name="${prefix}laser">
     <visual>
       <geometry>
@@ -90,11 +91,11 @@
     </visual>
   </link>
-  <joint name="base_laser" type="fixed">
-    <parent link="base_link"/>
-    <child link="laser"/>
+  <joint name="${prefix}base_laser" type="fixed">
+    <parent link="${prefix}base_link"/>
+    <child link="${prefix}laser"/>
     <origin xyz="${width} 0 ${GROUND_CLEARANCE-bodylen+posz_laser} " rpy="0 0 0"/>
   </joint>
   <!--FRONT WHEEL-->
-  <link name="fwheel">
+  <link name="${prefix}fwheel">
     <visual>
       <geometry>
@@ -111,12 +112,12 @@
     </collsion>
   </link>
-  <joint name="base_to_fwheel" type="continuous">
-    <parent link="base_link"/>
-    <child link="fwheel"/>
+  <joint name="${prefix}base_to_fwheel" type="continuous">
+    <parent link="${prefix}base_link"/>
+    <child link="${prefix}fwheel"/>
     <axis xyz="0 1 0"/>
     <origin xyz="${width} 0 ${GROUND_CLEARANCE-(bodylen/2)-(fwheel_rad)}" rpy="0 0 0"/>
   </joint>
   <!--BACK WHEEL-->
-  <link name="bwheel">
+  <link name="${prefix}bwheel">
     <visual>
       <geometry>
@@ -133,12 +134,12 @@
     </collsion>
   </link>
-  <joint name="base_to_bwheel" type="continuous">
-    <parent link="base_link"/>
-    <child link="bwheel"/>
+  <joint name="${prefix}base_to_bwheel" type="continuous">
+    <parent link="${prefix}base_link"/>
+    <child link="${prefix}bwheel"/>
     <axis xyz="0 1 0"/>
     <origin xyz="${-width} 0 ${GROUND_CLEARANCE-(bodylen/2)-(fwheel_rad)}" rpy="0 0 0"/>
   </joint>
   <!-- PLatform qui se leve-->
-  <link name="platform">
+  <link name="${prefix}platform">
     <visual>
       <geometry>
@@ -149,7 +150,7 @@
     </visual>
   </link>
-  <joint name="base_platform" type="prismatic">
-    <parent link="base_link"/>
-    <child link="platform"/>
+  <joint name="${prefix}base_platform" type="prismatic">
+    <parent link="${prefix}base_link"/>
+    <child link="${prefix}platform"/>
     <axis xyz="0 0 1"/>
     <limit effort="1000.0" lower="0" upper="${HIGH_PLATFORM}" velocity="0.5"/>
@@ -157,5 +158,5 @@
   </joint>
   <!--CAMERA-->
-  <link name="camera_link">
+  <link name="${prefix}camera_link">
     <visual>
       <geometry>
@@ -166,7 +167,7 @@
     </visual>
   </link>
-  <joint name="camera_link" type="fixed">
-    <parent link="base_link"/>
-    <child link="camera_link"/>
+  <joint name="${prefix}camera_link" type="fixed">
+    <parent link="${prefix}base_link"/>
+    <child link="${prefix}camera_link"/>
     <origin xyz="${width} 0 ${GROUND_CLEARANCE-bodylen+posz_camera} " rpy="${-PI/2} 0 ${-PI/2}"/>
   </joint>

Commit message: Upadet URDF

File: simulation_tobot/URDF/tobot.urdf.xacro (robot description, xacro)
@@ -2,13 +2,14 @@
 <robot xmlns:xacro="http://www.ros.org/wiki/xacro" name="tobot">
   <!-- Constant for the xacro model -->
-  <xacro:property name="GROUND_CLEARANCE" value="0.2" />
-  <xacro:property name="width" value="0.285" />
+  <xacro:property name="GROUND_CLEARANCE" value="0.0938" />
+  <xacro:property name="width" value="0.2102" />
   <xacro:property name="bodylen" value="0.355" />
   <xacro:property name="wheel_w" value="0.039" />
-  <xacro:property name="wheel_rad" value="0.075" />
-  <xacro:property name="plat_rad" value="0.285" />
+  <xacro:property name="wheel_rad" value="0.0938" />
+  <xacro:property name="plat_rad" value="0.150" />
   <xacro:property name="plat_len" value="0.005" />
   <xacro:property name="HIGH_PLATFORM" value="0.15" />
-  <xacro:property name="posz_laser" value="0.285" />
+  <xacro:property name="posz_laser" value="0.280" />
+  <xacro:property name="posx_laser" value="0.385" />
   <xacro:property name="posz_camera" value="0.5" />
   <xacro:property name="fwheel_rad" value="0.0325" />
@@ -94,5 +95,5 @@
     <parent link="${prefix}base_link"/>
     <child link="${prefix}laser"/>
-    <origin xyz="${width} 0 ${GROUND_CLEARANCE-bodylen+posz_laser} " rpy="0 0 0"/>
+    <origin xyz="${GROUND_CLEARANCE-posx_laser} 0 ${GROUND_CLEARANCE-posx_laser+posz_laser} " rpy="0 0 0"/>
   </joint>
   <!--FRONT WHEEL-->

Commit message: Changed parameters and correct the weird rpm calculation...

File: simulation_tobot/URDF/tobot.urdf.xacro (robot description, xacro)
@@ -5,5 +5,5 @@
   <xacro:property name="width" value="0.2102" />
   <xacro:property name="bodylen" value="0.355" />
-  <xacro:property name="wheel_w" value="0.039" />
+  <xacro:property name="wheel_l" value="0.039" />
   <xacro:property name="wheel_rad" value="0.0938" />
   <xacro:property name="plat_rad" value="0.150" />
@@ -43,5 +43,5 @@
     <visual>
       <geometry>
-        <cylinder length="${wheel_w}" radius="${wheel_rad}"/>
+        <cylinder length="${wheel_l}" radius="${wheel_rad}"/>
       </geometry>
       <origin rpy="-1.57075 0 0" xyz="0 0 0"/>
@@ -50,5 +50,5 @@
     <collsion>
       <geometry>
-        <cylinder length="${wheel_w}" radius="${wheel_rad}"/>
+        <cylinder length="${wheel_l}" radius="${wheel_rad}"/>
       </geometry>
       <origin rpy="-1.57075 0 0" xyz="0 0 0"/>
@@ -64,5 +64,5 @@
     <visual>
       <geometry>
-        <cylinder length="${wheel_w}" radius="${wheel_rad}"/>
+        <cylinder length="${wheel_l}" radius="${wheel_rad}"/>
       </geometry>
       <origin rpy="-1.57075 0 0" xyz="0 0 0"/>
@@ -71,5 +71,5 @@
     <collsion>
       <geometry>
-        <cylinder length="${wheel_w}" radius="${wheel_rad}"/>
+        <cylinder length="${wheel_l}" radius="${wheel_rad}"/>
       </geometry>
       <origin rpy="-1.57075 0 0" xyz="0 0 0"/>
@@ -101,5 +101,5 @@
     <visual>
       <geometry>
-        <cylinder length="${wheel_w}" radius="${fwheel_rad}"/>
+        <cylinder length="${wheel_l}" radius="${fwheel_rad}"/>
       </geometry>
       <origin rpy="-1.57075 0 0" xyz="0 0 0"/>
@@ -108,5 +108,5 @@
     <collsion>
       <geometry>
-        <cylinder length="${wheel_w}" radius="${fwheel_rad}"/>
+        <cylinder length="${wheel_l}" radius="${fwheel_rad}"/>
       </geometry>
       <origin rpy="-1.57075 0 0" xyz="0 0 0"/>
@@ -123,5 +123,5 @@
     <visual>
       <geometry>
-        <cylinder length="${wheel_w}" radius="${fwheel_rad}"/>
+        <cylinder length="${wheel_l}" radius="${fwheel_rad}"/>
       </geometry>
       <origin rpy="-1.57075 0 0" xyz="0 0 0"/>
@@ -130,5 +130,5 @@
     <collsion>
       <geometry>
-        <cylinder length="${wheel_w}" radius="${fwheel_rad}"/>
+        <cylinder length="${wheel_l}" radius="${fwheel_rad}"/>
       </geometry>
       <origin rpy="-1.57075 0 0" xyz="0 0 0"/>

Commit message: Change move_base parameters, add better odometry and reading function. Not fast enough to provide the odometry though

File: simulation_tobot/URDF/tobot.urdf.xacro (robot description, xacro)
@@ -3,8 +3,8 @@
   <!-- Constant for the xacro model -->
   <xacro:property name="GROUND_CLEARANCE" value="0.0938" />
-  <xacro:property name="width" value="0.2102" />
+  <xacro:property name="width" value="0.30" />
   <xacro:property name="bodylen" value="0.355" />
   <xacro:property name="wheel_l" value="0.039" />
-  <xacro:property name="wheel_rad" value="0.0938" />
+  <xacro:property name="wheel_rad" value="0.0750" />
   <xacro:property name="plat_rad" value="0.150" />
   <xacro:property name="plat_len" value="0.005" />
@@ -171,5 +171,5 @@
     <parent link="${prefix}base_link"/>
     <child link="${prefix}camera_link"/>
-    <origin xyz="${width} 0 ${GROUND_CLEARANCE-bodylen+posz_camera} " rpy="${-PI/2} 0 ${-PI/2}"/>
+    <origin xyz="${width} 0 ${GROUND_CLEARANCE-bodylen+posz_camera} " rpy="0 0 0"/>
   </joint>
 </robot>

Commit message: Added TODO since we need to make sure that the bounding box is in the same coordinate frame than the point cloud.

File: simulation_tobot/URDF/tobot.urdf.xacro (robot description, xacro)
@@ -2,6 +2,6 @@
 <robot xmlns:xacro="http://www.ros.org/wiki/xacro" name="tobot">
   <!-- Constant for the xacro model -->
-  <xacro:property name="GROUND_CLEARANCE" value="0.0938" />
-  <xacro:property name="width" value="0.30" />
+  <xacro:property name="GROUND_CLEARANCE" value="0" />
+  <xacro:property name="width" value="0.20" />
   <xacro:property name="bodylen" value="0.355" />
   <xacro:property name="wheel_l" value="0.039" />
@@ -10,7 +10,7 @@
   <xacro:property name="plat_len" value="0.005" />
   <xacro:property name="HIGH_PLATFORM" value="0.15" />
-  <xacro:property name="posz_laser" value="0.280" />
-  <xacro:property name="posx_laser" value="0.385" />
-  <xacro:property name="posz_camera" value="0.5" />
+  <xacro:property name="posz_laser" value="0.12" />
+  <xacro:property name="posx_laser" value="0.15" />
+  <xacro:property name="posz_camera" value="0.2" />
   <xacro:property name="fwheel_rad" value="0.0325" />
   <xacro:property name="PI" value="3.1415" />
@@ -37,5 +37,5 @@
          <cylinder length="${bodylen}" radius="${width}"/>
       </geometry>
-      <origin rpy="0 0 0" xyz="0 0 ${bodylen/2}"/>
+      <origin rpy="0 0 0" xyz="0 0 ${GROUND_CLEARANCE+bodylen}"/>
     </collision>
   </link>
@@ -95,5 +95,5 @@
     <parent link="${prefix}base_link"/>
     <child link="${prefix}laser"/>
-    <origin xyz="${GROUND_CLEARANCE-posx_laser} 0 ${GROUND_CLEARANCE-posx_laser+posz_laser} " rpy="0 0 0"/>
+    <origin xyz="${width} 0 ${GROUND_CLEARANCE-(bodylen/2)+posz_laser} " rpy="0 0 0"/>
   </joint>
   <!--FRONT WHEEL-->
@@ -171,5 +171,5 @@
     <parent link="${prefix}base_link"/>
     <child link="${prefix}camera_link"/>
-    <origin xyz="${width} 0 ${GROUND_CLEARANCE-bodylen+posz_camera} " rpy="0 0 0"/>
+    <origin xyz="${width} 0 ${GROUND_CLEARANCE-(bodylen/2)+posz_camera} " rpy="0 0 0"/>
   </joint>
 </robot>
